File: Z88 EPROM KiCad/XavSnap EPROM v1.5.kicad_pcb (KiCad board)
At the start: 2 copper layers, 50.5 x 53.3 mm, 5 parts, among them J1 Conn_Z88, U1 NEC_ROM

Commit message: .
Routing:
- net /WEL: track 45.6 -> 43.8 mm
- net /A13: track 46.8 -> 45.3 mm
- net /A16: track 68.2 -> 67.4 mm
