File: Z88 EPROM KiCad/Z88 EPROM.kicad_pcb (KiCad board)
At the start: 2 copper layers, 50.5 x 53.3 mm, 5 parts, among them J1 Conn_Z88, U1 NEC_ROM

Commit message: cleanup
Routing:
- net /A0: track 34.3 -> 35.4 mm
- net /A3: track 29.2 -> 30.3 mm
- net /A1: track 32.5 -> 33.6 mm
- net /A2: track 30.9 -> 31.9 mm
- net /A4: track 27.6 -> 28.6 mm
- net /A5: track 25.9 -> 26.9 mm
- net /A6: track 24.3 -> 25.2 mm
- net /D1: track 37.8 -> 38.4 mm
- net /D2: track 40.0 -> 40.7 mm
- net /D0: track 35.5 -> 36.1 mm
Other:
- board text added: "Z88 128k EPROM Card"
- board text added: "https://github.com/markaudacity/Z88-EPROM-Card"
- board text removed: "Kicad released"
- board text removed: "Z88 - ROM Expansion"
- board text removed: "from XavSnap."

Commit message: simplified version
Parts:
- J1: footprint Z88:Conn_Z88_1.25mm -> Z88:Z88_Card_BONDED PADS
- JP1: value SolderJumper-3_P1.3mm_Bridged12_RoundedPad1.0x1.5mm -> NEC/JEDEC
- JP2: value SolderJumper-3_RoundedPad1.0x1.5mm -> NEC/JEDEC
Connections:
- JP1 pad 1: /ROE -> Net-(U1-A16)
- JP1 pad 2: /ROE -> /A16
- JP1 pad 3: /A16 -> Net-(U1-ROE)
- JP2 pad 1: /A16 -> Net-(U1-ROE)
- JP2 pad 2: /A16 -> /ROE
- JP2 pad 3: /ROE -> Net-(U1-A16)
- U1 pad 2: /A16 -> Net-(U1-ROE)
- U1 pad 24: /ROE -> Net-(U1-A16)
Routing:
- net GND: track 67.2 -> 6.25 mm
- net /ROE: track 91.5 -> 58.8 mm, vias 4 -> 2
- net Net-(U1-A16): track 0.00 -> 32.7 mm, vias 0 -> 2
- net /A16: track 67.4 -> 36.6 mm, vias 2 -> 0
- net Net-(U1-ROE): track 0.00 -> 30.8 mm, vias 0 -> 2
- net VCC: track 57.6 -> 54.5 mm
