File: Z88 EPROM Card simplified/Z88 EPROM Card simplified.kicad_sch (KiCad schematic)
At the start: 5 parts, among them J1 Conn_Z88, U1 27C100 (mask compatible)

Commit message: simplified version
Parts:
- removed JP1, JP2: NEC/JEDEC, Connector_PinHeader_2.54mm:Jumper_PinHeader_1x03_P2.54mm_Vertical, symbol Device:Jumper_NC_Dual
- removed U1: 27C100 (mask compatible), Package_DIP:DIP-32_W15.24mm, symbol Memory_EPROM_Custom:27C100
- added U3: 27C010, Package_DIP:DIP-32_W15.24mm_LongPads, symbol Memory_EPROM:27C010
- J1: symbol Z88:Z88_Card -> Z88:Conn_Z88
Connections:
- net A0: now also U3.12 (A0)
- net A1: now also U3.11 (A1)
- net A10: now also U3.23 (A10)
- net A11: now also U3.25 (A11)
- net A12: now also U3.4 (A12)
- net A13: now also U3.28 (A13)
- net A14: now also U3.29 (A14)
- net A15: now also U3.3 (A15)
- net A16: now also U3.2 (A16)
- net A2: now also U3.10 (A2)
- net A3: now also U3.9 (A3)
- net A4: now also U3.8 (A4)
- net A5: now also U3.7 (A5)
- net A6: now also U3.6 (A6)
- net A7: now also U3.5 (A7)
- net A8: now also U3.27 (A8)
- net A9: now also U3.26 (A9)
- net D0: now also U3.13 (D0)
- net D1: now also U3.14 (D1)
- net D2: now also U3.15 (D2)
- net D3: now also U3.17 (D3)
- net D4: now also U3.18 (D4)
- net D5: now also U3.19 (D5)
- net D6: now also U3.20 (D6)
- net D7: now also U3.21 (D7)
- net GND: now also C1.2, U3.16 (GND); no longer C1.1
- net VCC: now also C1.1, U3.32 (VCC); no longer C1.2
- net ~{CE}: now also U3.22 (~{CE})
- net ROE renamed ~{OE}
- net ~{OE}: now also U3.24 (~{OE})
- net Vpp renamed VPP
- net VPP: now also U3.1 (VPP)
- net WEL renamed ~{PGM}
- net ~{PGM}: now also U3.31 (~{PGM})
Other:
- note removed: "From https://worldofspectrum.org/z88forever/tech/hardware.htm"
- note removed: "Slot RAM/ROM RAM/ROM Eprom pins Slot 1 Slot 2 Slot 3 32K 128K 32K EPROM EPROM RAM 1 A16 A16 A16 - 24 - 2 A15 A15 A15 - 3 - 3 A12 A12 A12 2 4 2 4 A7 A7 A7 3 5 3 5 A6 A6 A6 4 6 4 6 A5 A5 A5 5 7 5 7 A4 A4 A4 6 8 6 8 A3 A3 A3 7 9 7 9 A2 A2 A2 8 10 8 10 A1 A1 A1 9 11 9 11 A0 A0 A0 10 12 10 12 D0 D0 D0 11 13 11 13 D1 D1 D1 12 14 12 14 D2 D2 D2 13 15 13 15 SNSL SNSL SNSL - - - 16 GND GND GND 14 16 14 17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"
- moved on the sheet: C1, J1
